File: hardware/W5500_PA_PTT_Control/kicad/w5500-esp32.kicad_sch (KiCad schematic)
At the start: 22 parts, among them J1 ESP32_DevKitC_Socket_40P_25.4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, J2 DC_IN_13V8, J5 Power, J6 PTT_ON, Q1 2SC1815, Q3 2SC1815, Q5 2SJ334, U1 TA48033S, U2 L7805

Commit message: PA/PTTコントローラの基板・資料をPi5版のRev.2.6に更新し、READMEに説明を追加
KiCadデータ・JLCPCB発注データ・日英併記の仕様書と接続一覧(Windows版の連携に
合わせて4.4節を記述)を入れ、READMEに日英併記の節を追加した。

Co-Authored-By: Claude Opus 5.5 <noreply@anthropic.com>
Parts:
- removed D1: LED_Red_3mm, LED_THT:LED_D3.0mm, symbol Device:LED
- removed D2: LED_Green_3mm, LED_THT:LED_D3.0mm, symbol Device:LED
- added J7: LED_PWR, Connector_JST:JST_XH_B2B-XH-A_1x02_P2.50mm_Vertical, symbol Connector_Generic:Conn_01x02
- added J8: LED_12V, Connector_JST:JST_XH_B2B-XH-A_1x02_P2.50mm_Vertical, symbol Connector_Generic:Conn_01x02
- added R12, R13: 10k, Resistor_THT:R_Axial_DIN0207_L6.3mm_D2.5mm_P5.08mm_Vertical, symbol Device:R
- A1: footprint project_footprints:W5500_Lite_2x06_P2.54mm_15.24mm -> project_footprints:W5500_Lite_USR-ES1_2x06_P2.54mm_20.32mm
- C1, C3: value 0.1uF -> 0.33uF
- C2: value 0.1uF -> 33uF
- J2, J5: footprint (none) -> Connector_Wire:SolderWire-1sqmm_1x02_P5.4mm_D1.4mm_OD2.7mm
- J6: footprint (none) -> Connector_JST:JST_XH_B2B-XH-A_1x02_P2.50mm_Vertical
- Q1, Q3: footprint Package_TO_SOT_THT:TO-92_Inline -> Package_TO_SOT_THT:TO-92_Inline_Wide
- Q5: symbol Device:Q_PMOS -> project_symbols:2SJ334
- R8: footprint Resistor_THT:R_Axial_DIN0207_L6.3mm_D2.5mm_P5.08mm_Vertical -> Resistor_THT:R_Axial_DIN0309_L9.0mm_D3.2mm_P5.08mm_Vertical
Connections:
- net +12V: now also Q5.3 (S); no longer Q5.S
- net GND: now also C1.2, C2.2, J1.21 (GND), J1.22 (GND), J1.23 (GND), J1.24 (GND), J1.40 (GND), J1.7 (GND), J2.2 (Pin_2), J5.2 (Pin_2), MCU1.7 (GND), Q1.1 (E), Q3.1 (E), U1.3 (GND), U2.2 (GND), J7.2 (Pin_2), J8.2 (Pin_2), R12.2, R13.2
- net Power: now also Q5.2 (D); no longer Q5.D
- net at R11.2: now also J8.1 (Pin_1)
- net at R10.2: now also J7.1 (Pin_1)
- net at Q1.2 (C), R8.1: now also Q5.1 (G); no longer Q5.G
- net at Q1.3 (B), R6.2: now also R12.1
- net at Q3.3 (B), R7.2: now also R13.1
- no-connect marks 60 -> 55
Other:
- note added: "U2: 13.8V(+12V)を5VへLDO変換(L7805)。発熱(13.8V-5V)*0.2A=約1.76Wのため放熱器を使用。 U1: 上記5VをさらにW5500(A1)専用の+3V3_Aへ変換(TA48033S)。発熱(5V-3.3V)*0.2A=約0.34W。放熱器を使用。 放熱器: U1・U2・Q5とも秋月[105054] 20×20×25mm(20PB020-01025、15.8℃/W)。 ESP32側(J1の3V3、DevKitC基板のオンボードLDO経由)とは完全に独立した系統。"
- note removed: "U2: 13.8V(+12V)を5VへLDO変換(L7805)。発熱(13.8V-5V)*0.2A=約1.76Wのためヒートシンク推奨。 U1: 上記5VをさらにW5500(A1)専用の+3V3_Aへ変換(TA48033S)。発熱(5V-3.3V)*0.2A=約0.34W。 ESP32側(J1の3V3、DevKitC基板のオンボードLDO経由)とは完全に独立した系統。"
